Commit message: fix(sim): turn the task scene the right way up, colour the models, size the gripper
Three corrections from the first Gazebo look.

Orientation.  The assembly frame is now turned 180 degrees about world Y, which
fixes two independent errors at once.  The module's handles sit on its own -Y
face, and -Y maps to assembly +X, so with the previous identity placement the
handles faced away from the robot; now the fixture opens toward the base.  And
assembly +Z points down, so the seated module used to protrude 19.3 mm BELOW the
fixture, i.e. through the floor; it now protrudes 19.3 mm above the fixture top,
which is what an inserted module does.  The fixture also sits directly on the
ground now, so the 40 mm stand-off is gone.

Materials.  Both task models and the ground carry explicit diffuse colours.  A
white-on-white render made it impossible to tell whether the wedge slot had
survived, which is the one thing the first run had to answer.

Gripper.  The existing application gripper is kept rather than replaced, which
removes the flange-transform blocker: its kinematics are already correct (finger
axes 0 -1 0 and 0 1 0 move apart, i.e. the expanding brace) and it is already
mounted on the arm.  Its mass was the placeholder 0.33 kg against the measured
4.580 kg for 夹持机构0228; the links now sum to 4.580 kg.  The link geometry stays
a placeholder, and the comment says so, because the tool's support arms span
246.57 mm while these fingers reach only +/-58 mm.

File: src/cs625_ap_description/urdf/cs625_parallel_gripper.xacro (robot description, xacro)
@@ -2,7 +2,15 @@
 <robot xmlns:xacro="http://www.ros.org/wiki/xacro">
   <!--
-    Simulation-only parallel gripper.  This is an application extension: it
-    never edits the Elite CS625 underlay.  The right finger is commanded by
-    gz_ros2_control and the left finger is a URDF mimic joint.
+    Simulation-only gripper.  This is an application extension: it never edits
+    the Elite CS625 underlay.  The right finger is commanded by gz_ros2_control
+    and the left finger is a URDF mimic joint.
+    The kinematics are right and are reused: both finger axes point away from the
+    tool axis, so the fingers move APART, which is the expanding brace the task
+    uses.  The scale is NOT right.  The real tool is 夹持机构0228, measured at
+    4.580 kg with a support-arm span of 246.57 mm, against a placeholder here of
+    0.33 kg whose fingers reach only +/-58 mm.  Masses and inertias below are set
+    from the measured tool; the link geometry stays a placeholder until the
+    transform from the tool's part frame to tool0 is known.  See
+    docs/real_hardware_readiness.md and config/cs625_task_scene.yaml.
   -->
   <xacro:macro name="cs625_parallel_gripper" params="parent prefix">
@@ -10,5 +18,6 @@
       <visual><geometry><box size="0.080 0.090 0.050"/></geometry><material name="gripper_dark"><color rgba="0.18 0.18 0.18 1"/></material></visual>
       <collision><geometry><box size="0.080 0.090 0.050"/></geometry></collision>
-      <inertial><mass value="0.25"/><inertia ixx="0.00020" ixy="0" ixz="0" iyy="0.00017" iyz="0" izz="0.00028"/></inertial>
+      <inertial><mass value="4.20"/><inertia ixx="0.00336" ixy="0" ixz="0" iyy="0.00286" iyz="0" izz="0.00470"/></inertial>
+      <!-- 4.20 + 2 x 0.19 = 4.580 kg, the measured 夹持机构0228 mass. -->
     </link>
     <joint name="${prefix}tool0_to_gripper_base" type="fixed">
@@ -19,5 +28,5 @@
       <visual><origin xyz="0.045 0 0"/><geometry><box size="0.090 0.014 0.070"/></geometry><material name="gripper_finger"><color rgba="0.32 0.32 0.32 1"/></material></visual>
       <collision><origin xyz="0.045 0 0"/><geometry><box size="0.090 0.014 0.070"/></geometry></collision>
-      <inertial><origin xyz="0.045 0 0"/><mass value="0.04"/><inertia ixx="0.00002" ixy="0" ixz="0" iyy="0.00003" iyz="0" izz="0.00003"/></inertial>
+      <inertial><origin xyz="0.045 0 0"/><mass value="0.19"/><inertia ixx="0.000095" ixy="0" ixz="0" iyy="0.0001425" iyz="0" izz="0.0001425"/></inertial>
     </link>
     <joint name="${prefix}gripper_right_finger_joint" type="prismatic">
@@ -29,5 +38,5 @@
       <visual><origin xyz="0.045 0 0"/><geometry><box size="0.090 0.014 0.070"/></geometry><material name="gripper_finger_left"><color rgba="0.32 0.32 0.32 1"/></material></visual>
       <collision><origin xyz="0.045 0 0"/><geometry><box size="0.090 0.014 0.070"/></geometry></collision>
-      <inertial><origin xyz="0.045 0 0"/><mass value="0.04"/><inertia ixx="0.00002" ixy="0" ixz="0" iyy="0.00003" iyz="0" izz="0.00003"/></inertial>
+      <inertial><origin xyz="0.045 0 0"/><mass value="0.19"/><inertia ixx="0.000095" ixy="0" ixz="0" iyy="0.0001425" iyz="0" izz="0.0001425"/></inertial>
     </link>
     <joint name="${prefix}gripper_left_finger_joint" type="prismatic">
