Commit message: fix(description): delete the phantom gripper and camera boxes
The real tool is the mesh on my_end_effector_link (tool0_vision.STL for the
visual, tool0_collision.STL for collision); it carries both the gripper and the
camera.  Two placeholder bodies were drawing a second, phantom tool beside it:
a 0.080 x 0.090 x 0.050 palm with two 0.090 x 0.014 x 0.070 fingers in
cs625_parallel_gripper.xacro, and a 0.03 x 0.05 x 0.02 box in
cs625_camera_extension.xacro.  Both geometries are removed.

The links, the prismatic finger joints, the inertials and the ros2_control
entries stay, because four things name them and would break if they vanished:
the SRDF's disable_collisions pairs, sim_controllers.yaml driving
gripper_right_finger_joint, test/apply_task_fixture_scene.py's FINGER_LINKS, and
the payload budget.  The rgbd_camera sensor also stays: the whole RGB-D contract
hangs off camera_link and its optical frames.

Verified after the change: xacro still expands to 22 links and 21 joints, only
the arm meshes and my_end_effector_link carry geometry, both finger joints and
their ros2_control interfaces survive, contract_checks passes and the gripper
scene tests still pass.

Still placeholders and still wrong for this task, recorded rather than hidden:
the 0.353 m flange-to-eef offset and the camera mount extrinsics, and the finger
stroke, which is 0..0.040 m against a real brace that closes with 0.00257 m of
preload.

File: src/cs625_ap_description/urdf/cs625_camera_extension.xacro (robot description, xacro)
@@ -23,14 +23,14 @@
       <origin xyz="${xyz}" rpy="${rpy}"/>
     </joint>
+    <!-- The camera is part of the real tool mesh on my_end_effector_link
+         (tool0_vision.STL / tool0_collision.STL), so the 0.03 x 0.05 x 0.02 m
+         placeholder box that used to sit here was deleted: it drew a second,
+         phantom camera next to the real one.
+         The link itself is kept, and so is the rgbd_camera sensor below, because
+         the whole RGB-D contract hangs off camera_link and its optical frames.
+         Only the geometry is gone.  camera_mount_xyz / camera_mount_rpy in the
+         launch arguments still place this frame and are still placeholders; they
+         must be set from the real extrinsics before the sensor pose is trusted. -->
     <link name="${prefix}camera_link">
-      <visual>
-        <geometry><box size="0.03 0.05 0.02"/></geometry>
-        <material name="camera_body">
-          <color rgba="0.20 0.20 0.20 1.0"/>
-        </material>
-      </visual>
-      <collision>
-        <geometry><box size="0.03 0.05 0.02"/></geometry>
-      </collision>
       <inertial>
         <mass value="0.05"/>

File: src/cs625_ap_description/urdf/cs625_parallel_gripper.xacro (robot description, xacro)
@@ -2,20 +2,24 @@
 <robot xmlns:xacro="http://www.ros.org/wiki/xacro">
   <!--
-    Simulation-only gripper.  This is an application extension: it never edits
-    the Elite CS625 underlay.  The right finger is commanded by gz_ros2_control
-    and the left finger is a URDF mimic joint.
-    The kinematics are right and are reused: both finger axes point away from the
-    tool axis, so the fingers move APART, which is the expanding brace the task
-    uses.  The scale is NOT right.  The real tool is 夹持机构0228, measured at
-    4.580 kg with a support-arm span of 246.57 mm, against a placeholder here of
-    0.33 kg whose fingers reach only +/-58 mm.  Masses and inertias below are set
-    from the measured tool; the link geometry stays a placeholder until the
-    transform from the tool's part frame to tool0 is known.  See
-    docs/real_hardware_readiness.md and config/cs625_task_scene.yaml.
+    Application gripper FRAMES only.  This is an application extension: it never
+    edits the Elite CS625 underlay.
+    The box geometry that used to live here was a placeholder: a 0.080 x 0.090 x
+    0.050 palm with two 0.090 x 0.014 x 0.070 fingers.  It is not the real tool.
+    The real tool is the mesh on my_end_effector_link (tool0_vision.STL /
+    tool0_collision.STL), which carries both the gripper and the camera, so the
+    boxes were deleted to stop a phantom gripper floating next to the real one.
+    The links, the prismatic finger joints and the masses are KEPT on purpose:
+      - cs625_active_perception.srdf names these links in disable_collisions,
+      - sim_controllers.yaml drives gripper_right_finger_joint,
+      - test/apply_task_fixture_scene.py uses FINGER_LINKS by name,
+      - the payload budget counts this mass.
+    Removing the links would break all four, so only the geometry is gone.
+    Mass 4.20 + 2 x 0.19 = 4.580 kg matches the measured 夹持机构0228.  The
+    finger stroke below (0..0.040 m) is still a placeholder; the real tool braces
+    its handles with 0.00257 m of preload.  See config/cs625_task_scene.yaml.
   -->
   <xacro:macro name="cs625_parallel_gripper" params="parent prefix">
     <link name="${prefix}gripper_base_link">
-      <visual><geometry><box size="0.080 0.090 0.050"/></geometry><material name="gripper_dark"><color rgba="0.18 0.18 0.18 1"/></material></visual>
-      <collision><geometry><box size="0.080 0.090 0.050"/></geometry></collision>
+      <!-- placeholder box removed: 0.080 0.090 0.050 m -->
       <inertial><mass value="4.20"/><inertia ixx="0.00336" ixy="0" ixz="0" iyy="0.00286" iyz="0" izz="0.00470"/></inertial>
       <!-- 4.20 + 2 x 0.19 = 4.580 kg, the measured 夹持机构0228 mass. -->
@@ -26,6 +30,5 @@
     </joint>
     <link name="${prefix}gripper_right_finger_link">
-      <visual><origin xyz="0.045 0 0"/><geometry><box size="0.090 0.014 0.070"/></geometry><material name="gripper_finger"><color rgba="0.32 0.32 0.32 1"/></material></visual>
-      <collision><origin xyz="0.045 0 0"/><geometry><box size="0.090 0.014 0.070"/></geometry></collision>
+      <!-- placeholder box removed: 0.090 0.014 0.070 m -->
       <inertial><origin xyz="0.045 0 0"/><mass value="0.19"/><inertia ixx="0.000095" ixy="0" ixz="0" iyy="0.0001425" iyz="0" izz="0.0001425"/></inertial>
     </link>
@@ -36,6 +39,5 @@
     </joint>
     <link name="${prefix}gripper_left_finger_link">
-      <visual><origin xyz="0.045 0 0"/><geometry><box size="0.090 0.014 0.070"/></geometry><material name="gripper_finger_left"><color rgba="0.32 0.32 0.32 1"/></material></visual>
-      <collision><origin xyz="0.045 0 0"/><geometry><box size="0.090 0.014 0.070"/></geometry></collision>
+      <!-- placeholder box removed: 0.090 0.014 0.070 m -->
       <inertial><origin xyz="0.045 0 0"/><mass value="0.19"/><inertia ixx="0.000095" ixy="0" ixz="0" iyy="0.0001425" iyz="0" izz="0.0001425"/></inertial>
     </link>
