Commit message: feat: complete simulation active perception workflow

File: src/cs625_ap_description/urdf/cs625_active_perception.urdf.xacro (robot description, xacro)
@@ -31,4 +31,8 @@
        default. The ROS-facing name is assigned by the bridge profile. -->
   <xacro:arg name="camera_sensor_topic" default="/camera"/>
+  <xacro:arg name="camera_image_width" default="320"/>
+  <xacro:arg name="camera_image_height" default="240"/>
+  <xacro:arg name="camera_update_rate" default="10.0"/>
+  <xacro:arg name="camera_enabled" default="true"/>
   <xacro:arg name="simulation_controllers" default=""/>
   <xacro:arg name="headless_mode" default="false"/>
@@ -152,4 +156,8 @@
     optical_rpy="$(arg camera_optical_rpy)"
     sim_ignition="$(arg sim_ignition)"
-    camera_sensor_topic="$(arg camera_sensor_topic)"/>
+    camera_sensor_topic="$(arg camera_sensor_topic)"
+    camera_image_width="$(arg camera_image_width)"
+    camera_image_height="$(arg camera_image_height)"
+    camera_update_rate="$(arg camera_update_rate)"
+    camera_enabled="$(arg camera_enabled)"/>
 </robot>

File: src/cs625_ap_description/urdf/cs625_camera_extension.xacro (robot description, xacro)
@@ -7,5 +7,7 @@
   <xacro:macro name="cs625_eye_in_hand_camera"
                params="parent prefix xyz rpy optical_rpy
-                       sim_ignition:=false camera_sensor_topic:=/camera">
+                       sim_ignition:=false camera_sensor_topic:=/camera
+                       camera_image_width:=320 camera_image_height:=240
+                       camera_update_rate:=10.0 camera_enabled:=true">
     <link name="${prefix}camera_mount_link">
       <inertial>
@@ -31,4 +33,9 @@
         <geometry><box size="0.03 0.05 0.02"/></geometry>
       </collision>
+      <inertial>
+        <mass value="0.05"/>
+        <inertia ixx="0.00001" ixy="0" ixz="0"
+                 iyy="0.00001" iyz="0" izz="0.00001"/>
+      </inertial>
     </link>
     <joint name="${prefix}camera_mount_to_camera" type="fixed">
@@ -56,14 +63,16 @@
          stable /sim/camera/* names below the vendor boundary. -->
     <xacro:if value="${sim_ignition}">
-      <gazebo reference="${prefix}camera_link">
-        <sensor type="rgbd_camera" name="${prefix}camera_sensor">
+      <xacro:if value="${camera_enabled}">
+        <gazebo reference="${prefix}camera_link">
+          <sensor type="rgbd_camera" name="${prefix}camera_sensor">
+          <pose>0 0 0 0 0 0</pose>
           <always_on>1</always_on>
-          <update_rate>15.0</update_rate>
+          <update_rate>${camera_update_rate}</update_rate>
           <visualize>false</visualize>
           <camera>
             <horizontal_fov>1.047</horizontal_fov>
             <image>
-              <width>640</width>
-              <height>480</height>
+              <width>${camera_image_width}</width>
+              <height>${camera_image_height}</height>
               <format>R8G8B8</format>
             </image>
@@ -72,9 +81,10 @@
               <far>5.0</far>
             </clip>
+            <optical_frame_id>${prefix}camera_depth_optical_frame</optical_frame_id>
           </camera>
           <topic>${camera_sensor_topic}</topic>
-          <gz_frame_id>${prefix}camera_link</gz_frame_id>
-        </sensor>
-      </gazebo>
+          </sensor>
+        </gazebo>
+      </xacro:if>
     </xacro:if>
   </xacro:macro>

Commit message: feat: add P7 simulation gate evidence

File: src/cs625_ap_description/urdf/cs625_active_perception.urdf.xacro (robot description, xacro)
@@ -10,4 +10,5 @@
   <xacro:include filename="$(find eli_cs_robot_description)/urdf/cs_macro.xacro"/>
   <xacro:include filename="$(find cs625_ap_description)/urdf/cs625_camera_extension.xacro"/>
+  <xacro:include filename="$(find cs625_ap_description)/urdf/cs625_parallel_gripper.xacro"/>
   <xacro:arg name="name" default="cs625"/>
   <xacro:arg name="cs_type" default="cs625"/>
@@ -36,4 +37,5 @@
   <xacro:arg name="camera_enabled" default="true"/>
   <xacro:arg name="simulation_controllers" default=""/>
+  <xacro:arg name="p7_attachment_enabled" default="true"/>
   <xacro:arg name="headless_mode" default="false"/>
   <xacro:arg name="robot_ip" default="0.0.0.0"/>
@@ -52,5 +54,10 @@
   <xacro:arg name="tool_stop_bits" default="1"/>
   <xacro:arg name="tool_tcp_port" default="54321"/>
-  <xacro:arg name="camera_mount_xyz" default="0.05 0 0.05"/>
+  <!-- Mount the eye-in-hand camera above and slightly behind the gripper.
+       The old (0.05, 0, 0.05) pose placed the gripper palm about 60 mm along
+       the optical ray; P7.1 d1 proved that even a 160 mm marker at the target
+       was invisible.  At (0.03, 0, 0.15), the 45-degree centre ray clears the
+       palm's z=0.025 m upper face by at least 30 mm over its full x extent. -->
+  <xacro:arg name="camera_mount_xyz" default="0.03 0 0.15"/>
   <xacro:arg name="camera_mount_rpy" default="0 0.785398163397 0"/>
   <!-- camera_link uses the usual body convention; optical is x-right,
@@ -116,7 +123,49 @@
         <robot_param_node>robot_state_publisher</robot_param_node>
         <parameters>$(arg simulation_controllers)</parameters>
+        <!-- gz_ros2_control maps the position interface to a velocity
+             setpoint.  Its default 0.1 gain leaves the heavy CS625 fixture
+             materially behind a retimed P7 trajectory; 0.5 is within the
+             Jazzy documented non-oscillatory range (<= 1) and is simulation
+             only. -->
+        <position_proportional_gain>0.5</position_proportional_gain>
         <controller_manager_name>$(arg prefix)controller_manager</controller_manager_name>
       </plugin>
+      <!-- P7 attachment-assisted grasp mechanism.  Gazebo's official
+           DetachableJoint starts attached, so a P7 episode must explicitly
+           publish /p7/attachment/detach during reset and may only publish
+           /p7/attachment/attach after its geometric pre-grasp gate passes.
+           This is an attachment state, not evidence of frictional contact. -->
+      <xacro:if value="$(arg p7_attachment_enabled)">
+        <plugin filename="gz-sim-detachable-joint-system"
+                name="gz::sim::systems::DetachableJoint">
+        <!-- Gazebo collapses the fixed tool / gripper chain when converting
+             the URDF; wrist_3_link is the terminal non-lumped actuated link
+             that remains addressable in the running CS625 model. -->
+        <parent_link>$(arg prefix)wrist_3_link</parent_link>
+        <child_model>target_object</child_model>
+        <child_link>target_link</child_link>
+        <detach_topic>/p7/attachment/detach</detach_topic>
+        <attach_topic>/p7/attachment/attach</attach_topic>
+          <output_topic>/p7/attachment/state</output_topic>
+        </plugin>
+      </xacro:if>
     </gazebo>
+    <!-- P7 validates task geometry and controller/TF consistency, not
+         force-accurate robot dynamics.  Make the robot's own articulated
+         links gravity-free so a position command is not torque-saturated by
+         the synthetic arm mass.  The YCB target remains dynamic in the world
+         and the attachment mechanism is still explicitly labelled kinematic.
+         This never applies to a real-robot profile. -->
+    <gazebo reference="$(arg prefix)base_link"><gravity>false</gravity></gazebo>
+    <gazebo reference="$(arg prefix)shoulder_link"><gravity>false</gravity></gazebo>
+    <gazebo reference="$(arg prefix)upperarm_link"><gravity>false</gravity></gazebo>
+    <gazebo reference="$(arg prefix)forearm_link"><gravity>false</gravity></gazebo>
+    <gazebo reference="$(arg prefix)wrist_1_link"><gravity>false</gravity></gazebo>
+    <gazebo reference="$(arg prefix)wrist_2_link"><gravity>false</gravity></gazebo>
+    <gazebo reference="$(arg prefix)wrist_3_link"><gravity>false</gravity></gazebo>
+    <gazebo reference="$(arg prefix)my_end_effector_link"><gravity>false</gravity></gazebo>
+    <gazebo reference="$(arg prefix)gripper_base_link"><gravity>false</gravity></gazebo>
+    <gazebo reference="$(arg prefix)gripper_left_finger_link"><gravity>false</gravity></gazebo>
+    <gazebo reference="$(arg prefix)gripper_right_finger_link"><gravity>false</gravity></gazebo>
   </xacro:if>
   <!-- Preserved from the senior CS625 description so the existing MoveIt
@@ -149,4 +198,18 @@
     <origin xyz="0 0 0" rpy="0 0 0"/>
   </joint>
+  <xacro:cs625_parallel_gripper parent="$(arg prefix)tool0" prefix="$(arg prefix)"/>
+  <!-- Nominal cylindrical-object grasp centre between the two finger pads.
+       The pad volumes span x=0.005..0.095 m from gripper_base_link, while the
+       palm collision ends at x=0.040 m.  Placing the reference at x=0.080 m
+       leaves 6 mm clearance behind the 34 mm-radius tomato-can proxy; the old
+       pad-volume midpoint at x=0.050 m overlapped the palm and pushed the can.
+       The link is massless and collision-free and remains centred laterally
+       while the two prismatic fingers move symmetrically. -->
+  <link name="$(arg prefix)p7_grasp_center_link"/>
+  <joint name="$(arg prefix)gripper_base_to_p7_grasp_center" type="fixed">
+    <parent link="$(arg prefix)gripper_base_link"/>
+    <child link="$(arg prefix)p7_grasp_center_link"/>
+    <origin xyz="0.080 0 0" rpy="0 0 0"/>
+  </joint>
   <xacro:cs625_eye_in_hand_camera
     parent="$(arg prefix)tool0"

Commit message: feat(description): mount the real gripper on the flange
The tool owner exported 夹持机构0920.STL, the same rigid body as the earlier
0228 export but written directly in the FLANGE frame.  That removes the blocker
that has been open since the gripper was first measured.

The frame is confirmed from the geometry, not asserted: X is symmetric to
0.000 mm (-147.285..+147.285), and Z runs -7.0 mm, a locating boss behind the
mounting face, to +207.0 mm.  ICP against the 0228 export converges to
0.035 um median, 0.068 um max, every sample inside 1 um, so the two files are
the same body under an exact rigid transform and the new frame is trustworthy.

So my_end_effector_link now carries gripper_0920.stl with flange_to_eef_joint at
identity, and the old -0.046 0 0.353 offset is gone.  That offset was the
senior's: tool0_vision.STL is a different object, 177 x 240 x 214 mm against
294.6 x 85 x 214 mm, an ASCII mesh of 50 MB and 183373 triangles, sitting
146..360 mm off its own origin.  With the real tool the FK distance
flange->my_end_effector_link is 0.000 mm, down from 356.0 mm.

The inertial is the measured 4.580 kg with the SolidWorks positive-tensor output
converted at 1e-6 and rotated into the flange frame; the centre of mass lands at
X -0.10 mm, which the symmetry check predicts.  The placeholder gripper links
drop to 1 g so the tool is not counted twice.

The mesh is decimated 185896 -> 27883 triangles at a 0.0000% volume change and
lives in cs625_ap_description/meshes/tool/, which the package now installs.

SRDF tip, P7 contracts and the ros2_control entries are untouched: only geometry
and one fixed-joint origin changed.

File: src/cs625_ap_description/urdf/cs625_active_perception.urdf.xacro (robot description, xacro)
@@ -169,11 +169,23 @@
     <gazebo reference="$(arg prefix)gripper_right_finger_link"><gravity>false</gravity></gazebo>
   </xacro:if>
-  <!-- Preserved from the senior CS625 description so the existing MoveIt
-       SRDF group (tip=my_end_effector_link) remains usable. -->
+  <!-- The real tool, exported from SolidWorks in the FLANGE frame: the origin is
+       the mounting face, X is the gripper's symmetry axis, and +Z runs out along
+       the tool.  Two independent checks say so: X is symmetric to 0.000 mm
+       (-147.285 .. +147.285), and Z runs -7.0 mm (a locating boss behind the face)
+       to +207.0 mm.  The mesh is already in metres, so no scale attribute.
+       This replaces the senior's tool0_vision.STL, which was a DIFFERENT object
+       (177 x 240 x 214 mm against 294.6 x 85 x 214 mm), was an ASCII mesh of
+       50 MB with 183373 triangles, and sat 146..360 mm off its own origin, which
+       is where the old -0.046 0 0.353 joint offset came from.  The joint below is
+       therefore identity: the tool's own frame is the flange frame.
+       Inertia is the SolidWorks positive-tensor output, converted at 1e-6 and
+       rotated from the part frame into this one; the mass is the measured
+       4.580 kg.  The centre of mass X is -0.10 mm, which the symmetry check above
+       predicts.  The SRDF tip stays my_end_effector_link, so the group, the P7
+       contracts and the MoveIt configuration are untouched. -->
   <link name="$(arg prefix)my_end_effector_link">
     <visual>
       <geometry>
-        <mesh filename="file://$(find eli_cs_robot_description)/meshes/visual/tool0_vision.STL"
-              scale="0.001 0.001 0.001"/>
+        <mesh filename="file://$(find cs625_ap_description)/meshes/tool/gripper_0920.stl"/>
       </geometry>
       <material name="eef_color"><color rgba="0.75 0.75 0.75 1.0"/></material>
@@ -181,13 +193,18 @@
     <collision>
       <geometry>
-        <mesh filename="file://$(find eli_cs_robot_description)/meshes/visual/tool0_collision.STL"
-              scale="0.001 0.001 0.001"/>
+        <mesh filename="file://$(find cs625_ap_description)/meshes/tool/gripper_0920.stl"/>
       </geometry>
     </collision>
+    <inertial>
+      <origin xyz="-0.0001013 0.0140800 0.1095589" rpy="0 0 0"/>
+      <mass value="4.580"/>
+      <inertia ixx="1.656126300e-02" ixy="4.500000000e-07" ixz="4.718400000e-05"
+               iyy="3.412100900e-02" iyz="-6.521470000e-04" izz="2.090739800e-02"/>
+    </inertial>
   </link>
   <joint name="$(arg prefix)flange_to_eef_joint" type="fixed">
     <parent link="$(arg prefix)flange"/>
     <child link="$(arg prefix)my_end_effector_link"/>
-    <origin xyz="-0.046 0 0.353" rpy="0 0 0"/>
+    <origin xyz="0 0 0" rpy="0 0 0"/>
   </joint>
   <!-- Stable application frame used by the active-perception contract. -->

File: src/cs625_ap_description/urdf/cs625_parallel_gripper.xacro (robot description, xacro)
@@ -15,13 +15,16 @@
       - the payload budget counts this mass.
     Removing the links would break all four, so only the geometry is gone.
-    Mass 4.20 + 2 x 0.19 = 4.580 kg matches the measured 夹持机构0228.  The
-    finger stroke below (0..0.040 m) is still a placeholder; the real tool braces
-    its handles with 0.00257 m of preload.  See config/cs625_task_scene.yaml.
+    Masses here are 1 g placeholders.  The measured 4.580 kg of 夹持机构0228 now
+    lives on my_end_effector_link, where the real mesh is; leaving it here as well
+    would count the tool twice.  The finger stroke below (0..0.040 m) is still a
+    placeholder: the real tool braces its handles with 0.00257 m of preload.  See
+    config/cs625_task_scene.yaml.
   -->
   <xacro:macro name="cs625_parallel_gripper" params="parent prefix">
     <link name="${prefix}gripper_base_link">
       <!-- placeholder box removed: 0.080 0.090 0.050 m -->
-      <inertial><mass value="4.20"/><inertia ixx="0.00336" ixy="0" ixz="0" iyy="0.00286" iyz="0" izz="0.00470"/></inertial>
-      <!-- 4.20 + 2 x 0.19 = 4.580 kg, the measured 夹持机构0228 mass. -->
+      <inertial><mass value="0.001"/><inertia ixx="1e-9" ixy="0" ixz="0" iyy="1e-9" iyz="0" izz="1e-9"/></inertial>
+      <!-- Massless placeholder: the real 4.580 kg now sits on my_end_effector_link,
+           where the real mesh is.  Keeping it here too would double-count it. -->
     </link>
     <joint name="${prefix}tool0_to_gripper_base" type="fixed">
@@ -31,5 +34,5 @@
     <link name="${prefix}gripper_right_finger_link">
       <!-- placeholder box removed: 0.090 0.014 0.070 m -->
-      <inertial><origin xyz="0.045 0 0"/><mass value="0.19"/><inertia ixx="0.000095" ixy="0" ixz="0" iyy="0.0001425" iyz="0" izz="0.0001425"/></inertial>
+      <inertial><origin xyz="0.045 0 0"/><mass value="0.001"/><inertia ixx="1e-9" ixy="0" ixz="0" iyy="1e-9" iyz="0" izz="1e-9"/></inertial>
     </link>
     <joint name="${prefix}gripper_right_finger_joint" type="prismatic">
@@ -40,5 +43,5 @@
     <link name="${prefix}gripper_left_finger_link">
       <!-- placeholder box removed: 0.090 0.014 0.070 m -->
-      <inertial><origin xyz="0.045 0 0"/><mass value="0.19"/><inertia ixx="0.000095" ixy="0" ixz="0" iyy="0.0001425" iyz="0" izz="0.0001425"/></inertial>
+      <inertial><origin xyz="0.045 0 0"/><mass value="0.001"/><inertia ixx="1e-9" ixy="0" ixz="0" iyy="1e-9" iyz="0" izz="1e-9"/></inertial>
     </link>
     <joint name="${prefix}gripper_left_finger_joint" type="prismatic">
