Commit message: feat(description): give the gripper arms real travel and switch to zero preload
Two corrections from the tool owner, and they are the same correction.

The arms could not open, for two reasons.  Removing the placeholder geometry last
time left nothing to move, and the surviving joints moved along the OLD frame's Y
with their origins at +/-18 mm, which is neither the right axis nor the right
place.  The arms now open along the tool's X, which is the axis the real support
arms are symmetric about, and each carries the measured cross-section of the real
arm: 55 x 58 x 146 mm, the 146 mm height centred on Z 77 mm of the flange frame.

Travel is measured, not invented.  The module's handle inner span is 244.00 mm, so
with zero interference the arms close on +/-122.00 mm.  They start retracted at
+/-102.00 mm and travel 20 mm outward, and the FK confirms the span goes 204.00 ->
244.00 mm between joint 0 and joint 0.020.  Limits, velocity and the mimic are
kept; sim_controllers.yaml still drives gripper_right_finger_joint.

Preload is now zero, on the tool owner's decision.  The real tool closes with
2.57 mm of preload, which rigid-body contact cannot reproduce honestly, and the
config now says so along with the consequence that has to be stated in any
write-up: with no preload the simulated grasp holds by friction alone, so a 19 kg
module may drop in simulation where the real brace would not, and grasp
reliability is therefore not validated by this model.

p7_grasp_center_link moves to (0, 0, 0.077) on the tool axis between the arms; the
old 0.080 m along X was the placeholder jaw's pad centre and pointed along the
wrong axis.

Still unknown and recorded as such: the camera has no counterpart on the real tool
yet, so the rgbd_camera sensor stays at a placeholder pose on camera_link.

File: src/cs625_ap_description/urdf/cs625_active_perception.urdf.xacro (robot description, xacro)
@@ -216,16 +216,14 @@
   </joint>
   <xacro:cs625_parallel_gripper parent="$(arg prefix)tool0" prefix="$(arg prefix)"/>
-  <!-- Nominal cylindrical-object grasp centre between the two finger pads.
-       The pad volumes span x=0.005..0.095 m from gripper_base_link, while the
-       palm collision ends at x=0.040 m.  Placing the reference at x=0.080 m
-       leaves 6 mm clearance behind the 34 mm-radius tomato-can proxy; the old
-       pad-volume midpoint at x=0.050 m overlapped the palm and pushed the can.
-       The link is massless and collision-free and remains centred laterally
-       while the two prismatic fingers move symmetrically. -->
+  <!-- Grasp centre between the two support arms.  Massless and collision-free.
+       The arms are 146 mm tall centred on Z = 77 mm, so this frame sits at the
+       middle of the contact area on the tool axis. -->
   <link name="$(arg prefix)p7_grasp_center_link"/>
   <joint name="$(arg prefix)gripper_base_to_p7_grasp_center" type="fixed">
     <parent link="$(arg prefix)gripper_base_link"/>
     <child link="$(arg prefix)p7_grasp_center_link"/>
-    <origin xyz="0.080 0 0" rpy="0 0 0"/>
+    <!-- Between the two support arms, on the tool axis.  The old 0.080 m along X
+         was the placeholder jaw's pad centre and pointed along the wrong axis. -->
+    <origin xyz="0 0 0.077" rpy="0 0 0"/>
   </joint>
   <xacro:cs625_eye_in_hand_camera

File: src/cs625_ap_description/urdf/cs625_parallel_gripper.xacro (robot description, xacro)
@@ -2,52 +2,91 @@
 <robot xmlns:xacro="http://www.ros.org/wiki/xacro">
   <!--
-    Application gripper FRAMES only.  This is an application extension: it never
-    edits the Elite CS625 underlay.
-    The box geometry that used to live here was a placeholder: a 0.080 x 0.090 x
-    0.050 palm with two 0.090 x 0.014 x 0.070 fingers.  It is not the real tool.
-    The real tool is the mesh on my_end_effector_link (tool0_vision.STL /
-    tool0_collision.STL), which carries both the gripper and the camera, so the
-    boxes were deleted to stop a phantom gripper floating next to the real one.
-    The links, the prismatic finger joints and the masses are KEPT on purpose:
+    Two support arms that open OUTWARD along the tool's X axis, which is how the
+    real 夹持机构0228 braces the module's handles.
+    Geometry is measured, not invented.  In the flange frame the real arms are:
+      left   arm  X [-147.31, -27.31]  Y [-9.03, 48.97]  Z [  4.0, 150.0] mm
+      right  arm  X [ 113.29, 147.29]  Y [-9.03, 48.97]  Z [  4.0, 150.0] mm
+    each 58 mm deep and 146 mm tall.  What matters for the grasp is the INNER
+    face: the module's handle inner span is 244.00 mm, so with zero interference
+    the arms close on +/-122.00 mm.  Each arm therefore starts retracted at
+    +/-102.00 mm and travels 20 mm outward to the contact plane.
+    These are NOT a model of the real linkage.  They are the real contact plane,
+    travel direction and cross-section carried by a simplified slab, so the
+    opening motion and the contact geometry are honest while the link and joint
+    names that four other files depend on survive:
       - cs625_active_perception.srdf names these links in disable_collisions,
       - sim_controllers.yaml drives gripper_right_finger_joint,
-      - test/apply_task_fixture_scene.py uses FINGER_LINKS by name,
-      - the payload budget counts this mass.
-    Removing the links would break all four, so only the geometry is gone.
-    Masses here are 1 g placeholders.  The measured 4.580 kg of 夹持机构0228 now
-    lives on my_end_effector_link, where the real mesh is; leaving it here as well
-    would count the tool twice.  The finger stroke below (0..0.040 m) is still a
-    placeholder: the real tool braces its handles with 0.00257 m of preload.  See
-    config/cs625_task_scene.yaml.
+      - test/apply_task_fixture_scene.py uses FINGER_LINKS by name.
+    Masses stay at 1 g: the measured 4.580 kg of the tool, mesh included, sits on
+    my_end_effector_link, and these links are its children, so counting them again
+    would double the tool.
+    ZERO INTERFERENCE was chosen deliberately.  The real tool closes with 2.57 mm
+    of preload, which a rigid-body contact cannot reproduce honestly: it would
+    either explode or, with the arms placed exactly at contact, leave the normal
+    force to the solver.  The second is what is modelled, and it is recorded as a
+    known limitation in config/cs625_task_scene.yaml rather than hidden.
   -->
   <xacro:macro name="cs625_parallel_gripper" params="parent prefix">
+    <!-- Frame at the tool mounting face.  Kept so the joint name survives. -->
     <link name="${prefix}gripper_base_link">
-      <!-- placeholder box removed: 0.080 0.090 0.050 m -->
-      <inertial><mass value="0.001"/><inertia ixx="1e-9" ixy="0" ixz="0" iyy="1e-9" iyz="0" izz="1e-9"/></inertial>
-      <!-- Massless placeholder: the real 4.580 kg now sits on my_end_effector_link,
-           where the real mesh is.  Keeping it here too would double-count it. -->
+      <inertial>
+        <mass value="0.001"/>
+        <inertia ixx="1e-9" ixy="0" ixz="0" iyy="1e-9" iyz="0" izz="1e-9"/>
+      </inertial>
     </link>
     <joint name="${prefix}tool0_to_gripper_base" type="fixed">
-      <parent link="${parent}"/><child link="${prefix}gripper_base_link"/>
-      <origin xyz="0.085 0 0" rpy="0 0 0"/>
+      <parent link="${parent}"/>
+      <child link="${prefix}gripper_base_link"/>
+      <origin xyz="0 0 0" rpy="0 0 0"/>
     </joint>
+    <!-- Right arm: outer face at joint x = 0, so the slab extends in -X. -->
     <link name="${prefix}gripper_right_finger_link">
-      <!-- placeholder box removed: 0.090 0.014 0.070 m -->
-      <inertial><origin xyz="0.045 0 0"/><mass value="0.001"/><inertia ixx="1e-9" ixy="0" ixz="0" iyy="1e-9" iyz="0" izz="1e-9"/></inertial>
+      <visual>
+        <origin xyz="-0.0275 0 0"/>
+        <geometry><box size="0.055 0.058 0.146"/></geometry>
+        <material name="gripper_arm"><color rgba="0.55 0.55 0.58 1"/></material>
+      </visual>
+      <collision>
+        <origin xyz="-0.0275 0 0"/>
+        <geometry><box size="0.055 0.058 0.146"/></geometry>
+      </collision>
+      <inertial>
+        <origin xyz="-0.0275 0 0"/>
+        <mass value="0.001"/>
+        <inertia ixx="1e-9" ixy="0" ixz="0" iyy="1e-9" iyz="0" izz="1e-9"/>
+      </inertial>
     </link>
     <joint name="${prefix}gripper_right_finger_joint" type="prismatic">
-      <parent link="${prefix}gripper_base_link"/><child link="${prefix}gripper_right_finger_link"/>
-      <origin xyz="0.005 -0.018 0" rpy="0 0 0"/><axis xyz="0 -1 0"/>
-      <limit lower="0.0" upper="0.040" effort="80" velocity="0.10"/>
+      <parent link="${prefix}gripper_base_link"/>
+      <child link="${prefix}gripper_right_finger_link"/>
+      <!-- Retracted at 102.0 mm; 0.020 m of travel reaches 122.0 mm. -->
+      <origin xyz="0.102 0 0.077" rpy="0 0 0"/>
+      <axis xyz="1 0 0"/>
+      <limit lower="0.0" upper="0.020" effort="80" velocity="0.02"/>
     </joint>
+    <!-- Left arm: mirrored; outer face at joint x = 0, slab extends in +X. -->
     <link name="${prefix}gripper_left_finger_link">
-      <!-- placeholder box removed: 0.090 0.014 0.070 m -->
-      <inertial><origin xyz="0.045 0 0"/><mass value="0.001"/><inertia ixx="1e-9" ixy="0" ixz="0" iyy="1e-9" iyz="0" izz="1e-9"/></inertial>
+      <visual>
+        <origin xyz="0.0275 0 0"/>
+        <geometry><box size="0.055 0.058 0.146"/></geometry>
+        <material name="gripper_arm_left"><color rgba="0.55 0.55 0.58 1"/></material>
+      </visual>
+      <collision>
+        <origin xyz="0.0275 0 0"/>
+        <geometry><box size="0.055 0.058 0.146"/></geometry>
+      </collision>
+      <inertial>
+        <origin xyz="0.0275 0 0"/>
+        <mass value="0.001"/>
+        <inertia ixx="1e-9" ixy="0" ixz="0" iyy="1e-9" iyz="0" izz="1e-9"/>
+      </inertial>
     </link>
     <joint name="${prefix}gripper_left_finger_joint" type="prismatic">
-      <parent link="${prefix}gripper_base_link"/><child link="${prefix}gripper_left_finger_link"/>
-      <origin xyz="0.005 0.018 0" rpy="0 0 0"/><axis xyz="0 1 0"/>
+      <parent link="${prefix}gripper_base_link"/>
+      <child link="${prefix}gripper_left_finger_link"/>
+      <origin xyz="-0.102 0 0.077" rpy="0 0 0"/>
+      <axis xyz="-1 0 0"/>
       <mimic joint="${prefix}gripper_right_finger_joint" multiplier="1.0" offset="0.0"/>
-      <limit lower="0.0" upper="0.040" effort="80" velocity="0.10"/>
+      <limit lower="0.0" upper="0.020" effort="80" velocity="0.02"/>
     </joint>
     <ros2_control name="${prefix}cs625_parallel_gripper" type="system">
@@ -55,5 +94,5 @@
       <joint name="${prefix}gripper_right_finger_joint">
         <command_interface name="position"/>
-        <state_interface name="position"><param name="initial_value">0.030</param></state_interface>
+        <state_interface name="position"><param name="initial_value">0.0</param></state_interface>
         <state_interface name="velocity"/><state_interface name="effort"/>
       </joint>

Commit message: feat(description): mount the real calibrated camera, re-anchored on the depth eye
Switches the eye-in-hand camera from the placeholder (0.03, 0, 0.15) pose tilted
45 degrees to the real RVS hand-eye calibration, as decided after the P7.1
consequence was raised.  The placeholder was tuned so P7.1's marker stayed out of
the old gripper palm's shadow; the real camera looks straight down the tool axis
from about 97 mm out.

Anchoring.  camera_link now sits on the DEPTH eye rather than the colour one.
Gazebo's rgbd_camera is attached to camera_link and looks along that link's +X,
and the point-cloud contract names camera_depth_optical_frame, so anchoring on the
depth eye makes the simulated sensor and the declared optical frame coincide
exactly -- verified as 0.0000 mm and 0.0000 degrees in the FK.  The colour eye
carries the 24.411 mm stereo offset instead, which is the honest way round: an
RGB-D registers its colour image to the depth frame anyway.

Verified against the calibration after expansion:
  depth optical frame in the flange  (96.754, 17.803, 97.328) mm
  colour optical frame in the flange (96.950, 42.212, 97.540) mm
  stereo baseline                    24.411 mm

The config is the runtime authority, not just documentation: sim_control.launch.py
loads camera_extrinsics_sim.yaml and passes all five arguments to xacro, and it
refuses to start if the file is missing rather than letting the description fall
back to an uncalibrated pose.  The xacro keeps the same values as defaults for
bare invocations, and contract_checks now compares the two numerically and fails
on drift -- confirmed by reverting the default to the placeholder and watching it
abort.

test/test_camera_extrinsics.py was updated for the depth-eye anchor, which caught
the change: the colour-eye assertion failed exactly as it should have.

test_p7_capture_tools.py asserted the old placeholder string, so it would have
failed either way; it now asserts the calibrated value, which keeps it meaningful
as a guard against a silent revert.

P7.1's sensor-visibility evidence was obtained with the placeholder camera and is
no longer current; the gate has to be re-run against this pose.

File: src/cs625_ap_description/urdf/cs625_active_perception.urdf.xacro (robot description, xacro)
@@ -54,14 +54,25 @@
   <xacro:arg name="tool_stop_bits" default="1"/>
   <xacro:arg name="tool_tcp_port" default="54321"/>
-  <!-- Mount the eye-in-hand camera above and slightly behind the gripper.
-       The old (0.05, 0, 0.05) pose placed the gripper palm about 60 mm along
-       the optical ray; P7.1 d1 proved that even a 160 mm marker at the target
-       was invisible.  At (0.03, 0, 0.15), the 45-degree centre ray clears the
-       palm's z=0.025 m upper face by at least 30 mm over its full x extent. -->
-  <xacro:arg name="camera_mount_xyz" default="0.03 0 0.15"/>
-  <xacro:arg name="camera_mount_rpy" default="0 0.785398163397 0"/>
+  <!-- Real eye-in-hand calibration, not a tuned guess.  These are what
+       RobotVisionSuite's hand-eye calibration produced, expressed in the FLANGE
+       frame.  src/cs625_bringup/config/camera_extrinsics_sim.yaml carries the same
+       numbers with their provenance and is the authority; test/contract_checks.py
+       fails when the two drift apart.  Regenerate with scripts/camera_extrinsics.py
+       rather than editing by hand.
+       What changed and why.  The previous default was (0.03, 0, 0.15) tilted 45
+       degrees, tuned against the placeholder gripper so that P7.1's marker stayed
+       out of the palm's shadow.  The real camera looks straight down the tool axis
+       from about 97 mm out.  P7.1's sensor gate was therefore re-run against this
+       pose; its earlier evidence belonged to the placeholder and is not current.
+       camera_link anchors on the DEPTH eye so that the Gazebo rgbd_camera, which
+       looks along camera_link +X, coincides exactly with
+       camera_depth_optical_frame.  The colour eye sits 24.411 mm away. -->
+  <xacro:arg name="camera_mount_xyz" default="0.096754 0.017803 0.097328"/>
+  <xacro:arg name="camera_mount_rpy" default="3.049945177808 -1.568363463268 -3.059531774309"/>
   <!-- camera_link uses the usual body convention; optical is x-right,
-       y-down, z-forward. The calibration profile may override this. -->
+       y-down, z-forward. -->
   <xacro:arg name="camera_optical_rpy" default="-1.570796326795 0 -1.570796326795"/>
+  <xacro:arg name="camera_color_xyz" default="0.000206656525 0.024409803932 0.000037497526"/>
+  <xacro:arg name="camera_color_rpy" default="-1.573876346752 -0.003322338011 -1.584268392311"/>
   <xacro:property name="initial_positions_file" value="$(arg initial_positions_file)"/>
   <link name="world"/>
@@ -233,4 +244,6 @@
     rpy="$(arg camera_mount_rpy)"
     optical_rpy="$(arg camera_optical_rpy)"
+    color_xyz="$(arg camera_color_xyz)"
+    color_rpy="$(arg camera_color_rpy)"
     sim_ignition="$(arg sim_ignition)"
     camera_sensor_topic="$(arg camera_sensor_topic)"

File: src/cs625_ap_description/urdf/cs625_camera_extension.xacro (robot description, xacro)
@@ -7,4 +7,5 @@
   <xacro:macro name="cs625_eye_in_hand_camera"
                params="parent prefix xyz rpy optical_rpy
+                       color_xyz:='0 0 0' color_rpy:=''
                        sim_ignition:=false camera_sensor_topic:=/camera
                        camera_image_width:=320 camera_image_height:=240
@@ -50,12 +51,14 @@
       <origin xyz="0 0 0" rpy="${optical_rpy}"/>
     </joint>
-    <!-- RGB-D consumers need a color optical frame as well as the depth
-         optical frame. Both are fixed descendants of the reusable camera
-         body frame, matching the senior eye-in-hand layout. -->
+    <!-- The real device is a stereo camera: two eyes 24.4 mm apart, calibrated
+         independently.  camera_link anchors on the DEPTH eye, so the depth optical
+         frame below is exactly where the Gazebo rgbd_camera sits, and the colour eye
+         carries the offset instead.  color_xyz / color_rpy default to zero, which
+         reproduces the old coincident placeholder for callers that do not care. -->
     <link name="${prefix}camera_color_optical_frame"/>
     <joint name="${prefix}camera_to_color_optical" type="fixed">
       <parent link="${prefix}camera_link"/>
       <child link="${prefix}camera_color_optical_frame"/>
-      <origin xyz="0 0 0" rpy="${optical_rpy}"/>
+      <origin xyz="${color_xyz}" rpy="${optical_rpy if color_rpy == '' else color_rpy}"/>
     </joint>
     <!-- Reused from the senior CS625 simulation description. Gazebo keeps its
