Commit message: feat(task): six task modes, real-cell-aligned simulation, dual UI, experiment archive
This is the 2026-10-24 reorganisation.  It turns the staged P4/P5/P7 work into a
single task layer and rebuilds the simulation from real measurements.

Task layer (scripts/, no new ROS package):
- run_task.py: --scope {load,unload,full} x --mode {safe,efficient} x
  --world {real,sim}; merges config, enforces the environment gate, records and
  archives every real run.
- run_pick_and_place.py: observation prefixes (observe:<waypoint>), config-driven
  phase lists, speed bands (retreat/entry slow only at the workpiece handles),
  a sincere timeout (waits for the controller's own verdict, reports NO_MOTION
  with the robot state), multi-seed IK with a URDF joint-limit check, and tight
  clearance phases planned without collision checks (1 mm gap < mesh error).
- model_environment.py: measured tables/slot/workpiece -> runtime model + gate.
- experiment_recorder.py / archive_experiment.py: 20 Hz timeseries, phase marks,
  process frames, trimming, archive under $HOME + docs index.
- camera_mode.py / capture_process_images.py / fit_fixture_to_cloud.py.

Simulation rebuilt from measurements (docs/simulation.md):
- build_sim_world.py generates cs625_real_cell.sdf + scene yaml from the real
  environment model; the fixture is the real RVS geometry (median 4.95 mm between
  the mesh and the camera cloud), the old hand-made worlds are archived.
- apply_real_cell_scene.py publishes the measured collision bodies to MoveIt.
- camera: 1280x960, FOV from the real fx, 1 Hz, depth noise, rendered at the
  colour eye; fixture/workpiece/table placement all evidence-based.

UI: Qt panel (468x960 + independent camera window, flow/phase card, live plots,
palette-independent log) and an RViz2 panel (palette-aware, control self-check,
flow/phase from /task_state).

Docs: README/AGENTS rewritten, docs/source_authority.md (A/B/C grading),
docs/sim_fidelity.md (measured fidelity, not claims), old docs archived under
docs/archive/2026-10-24-pre-six-modes, old sim assets snapshotted under
~/cs625_legacy_sim_snapshot_20261024.

Verification: 205 unit tests, contract checks PASS, six modes plan-only
19/19 19/19 38/38 38/38 57/57 57/57 with the real fixture collision body.
No real-arm motion: the robot was unreachable (No route to host).

File: src/cs625_ap_description/urdf/cs625_active_perception.urdf.xacro (robot description, xacro)
@@ -32,7 +32,23 @@
        default. The ROS-facing name is assigned by the bridge profile. -->
   <xacro:arg name="camera_sensor_topic" default="/camera"/>
-  <xacro:arg name="camera_image_width" default="320"/>
-  <xacro:arg name="camera_image_height" default="240"/>
-  <xacro:arg name="camera_update_rate" default="10.0"/>
+  <!-- Real Percipio PS800-E1 intrinsics, read from /camera/color/camera_info on
+       the real cell (config/real/camera_intrinsics.json is the same data and is
+       the authority for the real profile).  Gazebo Harmonic puts <lens>
+       <intrinsics> straight into camera_info, so the simulated K is the measured
+       K instead of a number re-derived from a rounded horizontal FOV.
+       sim_base.launch.py declares the same values as launch arguments; these
+       defaults only serve a bare xacro invocation. -->
+  <xacro:arg name="camera_image_width" default="1280"/>
+  <xacro:arg name="camera_image_height" default="960"/>
+  <xacro:arg name="camera_update_rate" default="1.0"/>
+  <xacro:arg name="camera_horizontal_fov_deg" default="68.98"/>
+  <xacro:arg name="camera_fx" default="931.47"/>
+  <xacro:arg name="camera_fy" default="931.60"/>
+  <xacro:arg name="camera_cx" default="648.70"/>
+  <xacro:arg name="camera_cy" default="449.32"/>
+  <xacro:arg name="camera_clip_near" default="0.2"/>
+  <xacro:arg name="camera_clip_far" default="3.0"/>
+  <xacro:arg name="camera_noise_mean" default="0.0"/>
+  <xacro:arg name="camera_noise_stddev" default="0.003"/>
   <xacro:arg name="camera_enabled" default="true"/>
   <xacro:arg name="simulation_controllers" default=""/>
@@ -67,5 +83,13 @@
        camera_link anchors on the DEPTH eye so that the Gazebo rgbd_camera, which
        looks along camera_link +X, coincides exactly with
-       camera_depth_optical_frame.  The colour eye sits 24.411 mm away. -->
+       camera_depth_optical_frame.  The colour eye sits 24.411 mm away.
+       The two lines below are the DEPTH eye, i.e. camera_mount_xyz / _rpy in
+       camera_extrinsics_sim.yaml (the generator's output).  Do not swap them for
+       the colour eye (0.096950 0.042212 0.097540): camera_color_xyz already
+       carries the 24.411 mm stereo baseline, so moving camera_link to the colour
+       eye would put camera_color_optical_frame 24.4 mm past the colour lens and
+       the depth optical frame 24.4 mm off the depth lens.  The colour eye is
+       reached by composing camera_mount @ camera_color_xyz; that composition is
+       what equals T_flange_cam_color_optical in config/handeye/tcp_to_camera.json. -->
   <xacro:arg name="camera_mount_xyz" default="0.096754 0.017803 0.097328"/>
   <xacro:arg name="camera_mount_rpy" default="3.049945177808 -1.568363463268 -3.059531774309"/>
@@ -251,4 +275,13 @@
     camera_image_height="$(arg camera_image_height)"
     camera_update_rate="$(arg camera_update_rate)"
+    camera_horizontal_fov_deg="$(arg camera_horizontal_fov_deg)"
+    camera_fx="$(arg camera_fx)"
+    camera_fy="$(arg camera_fy)"
+    camera_cx="$(arg camera_cx)"
+    camera_cy="$(arg camera_cy)"
+    camera_clip_near="$(arg camera_clip_near)"
+    camera_clip_far="$(arg camera_clip_far)"
+    camera_noise_mean="$(arg camera_noise_mean)"
+    camera_noise_stddev="$(arg camera_noise_stddev)"
     camera_enabled="$(arg camera_enabled)"/>
 </robot>

File: src/cs625_ap_description/urdf/cs625_camera_extension.xacro (robot description, xacro)
@@ -9,12 +9,21 @@
                        color_xyz:='0 0 0' color_rpy:=''
                        sim_ignition:=false camera_sensor_topic:=/camera
-                       camera_image_width:=320 camera_image_height:=240
-                       camera_update_rate:=10.0 camera_enabled:=true">
+                       camera_image_width:=1280 camera_image_height:=960
+                       camera_update_rate:=1.0 camera_enabled:=true
+                       camera_horizontal_fov_deg:=68.98
+                       camera_fx:=931.47 camera_fy:=931.60
+                       camera_cx:=648.70 camera_cy:=449.32
+                       camera_clip_near:=0.2 camera_clip_far:=3.0
+                       camera_noise_mean:=0.0 camera_noise_stddev:=0.003">
     <link name="${prefix}camera_mount_link">
       <inertial>
-        <mass value="0.01"/>
+        <!-- ESTIMATED, needs CAD mass/CoG.  Not measured.  No datasheet weight
+             exists in this repository, so 0.010 kg is a 60 x 60 x 20 mm
+             mounting-plate estimate; the inertia is the solid-box value at
+             that envelope and the CoM is left at the mounting point. -->
+        <mass value="0.010"/>
         <origin xyz="0 0 0" rpy="0 0 0"/>
-        <inertia ixx="0.000001" ixy="0" ixz="0"
-                 iyy="0.000001" iyz="0" izz="0.000001"/>
+        <inertia ixx="3.33e-06" ixy="0" ixz="0"
+                 iyy="6.00e-06" iyz="0" izz="3.33e-06"/>
       </inertial>
     </link>
@@ -35,7 +44,16 @@
     <link name="${prefix}camera_link">
       <inertial>
-        <mass value="0.05"/>
-        <inertia ixx="0.00001" ixy="0" ixz="0"
-                 iyy="0.00001" iyz="0" izz="0.00001"/>
+        <!-- ESTIMATED, needs CAD mass/CoG.  Not measured.  The real depth eye is
+             part of the tool mesh on my_end_effector_link, so this mass is again
+             a bookkeeping duplicate, kept at 0.050 kg because that makes the
+             whole camera share 0.060 kg = camera_kg_placeholder in
+             config/cs625_task_scene.yaml.  No PS800-E1 datasheet weight exists
+             here, and a real GigE depth module is likely HEAVIER than this, so
+             treat 0.060 kg as a lower estimate, not a measurement.  Inertia is
+             the solid-box value for a 30 x 80 x 30 mm envelope; CoM assumed at
+             the lens centre, which is also unverified. -->
+        <mass value="0.050"/>
+        <inertia ixx="3.04e-05" ixy="0" ixz="0"
+                 iyy="7.50e-06" iyz="0" izz="3.04e-05"/>
       </inertial>
     </link>
@@ -69,10 +87,27 @@
         <gazebo reference="${prefix}camera_link">
           <sensor type="rgbd_camera" name="${prefix}camera_sensor">
-          <pose>0 0 0 0 0 0</pose>
+          <!-- Render where the real COLOUR eye is, not at camera_link (the depth
+               eye): the application back-projects with T_tcp_cam, which describes
+               the colour optical frame, and the real depth stream is registered to
+               the colour image (the driver runs depth_registration_enable:=true).
+               The 24.4 mm stereo baseline therefore stays in the geometry, not in
+               the render.
+               TRANSLATION ONLY.  Gazebo looks along the sensor frame +X, which is
+               camera_link +X (the tool axis).  color_rpy is the rotation of the
+               OPTICAL axes relative to camera_link, so using it here would point
+               the camera 90 deg sideways (its +X would become camera_link -Y).
+               The optical rotation belongs to the fixed joint below, not to the
+               sensor pose. -->
+          <pose>${color_xyz} 0 0 0</pose>
           <always_on>1</always_on>
           <update_rate>${camera_update_rate}</update_rate>
           <visualize>false</visualize>
           <camera>
-            <horizontal_fov>1.047</horizontal_fov>
+            <!-- 68.98 deg = 2*atan(640/931.47), the real horizontal FOV.  Kept for
+                 documentation and for readers of the SDF; the <lens><intrinsics>
+                 block below is what actually sets the projection matrix, so the
+                 simulated K is the measured K and not a number re-derived from a
+                 rounded FOV. -->
+            <horizontal_fov>${camera_horizontal_fov_deg * pi / 180.0}</horizontal_fov>
             <image>
               <width>${camera_image_width}</width>
@@ -81,8 +116,34 @@
             </image>
             <clip>
-              <near>0.05</near>
-              <far>5.0</far>
+              <!-- the real PS800-E1 is unusable closer than ~0.2 m and the task
+                   never looks further than 3 m -->
+              <near>${camera_clip_near}</near>
+              <far>${camera_clip_far}</far>
             </clip>
-            <optical_frame_id>${prefix}camera_depth_optical_frame</optical_frame_id>
+            <!-- Real depth is not synthetic-clean: metal parts come back with
+                 3-4 mm scatter and ~25 % holes.  3 mm Gaussian is the measured
+                 scatter; the holes are a rendering limitation we do not fake. -->
+            <noise>
+              <type>gaussian</type>
+              <mean>${camera_noise_mean}</mean>
+              <stddev>${camera_noise_stddev}</stddev>
+            </noise>
+            <!-- Measured Percipio PS800-E1 intrinsics at 1280x960; this is what
+                 Gazebo Harmonic copies into sensor_msgs/CameraInfo, so the bridge
+                 publishes the real K.  cx/cy are NOT the image centre: the real
+                 principal point sits 8.7 px right and 30.7 px above centre, and
+                 only an explicit intrinsics block reproduces that. -->
+            <lens>
+              <type>gnomonical</type>
+              <scale_to_hfov>true</scale_to_hfov>
+              <intrinsics>
+                <fx>${camera_fx}</fx>
+                <fy>${camera_fy}</fy>
+                <cx>${camera_cx}</cx>
+                <cy>${camera_cy}</cy>
+                <s>0.0</s>
+              </intrinsics>
+            </lens>
+            <optical_frame_id>${prefix}camera_color_optical_frame</optical_frame_id>
           </camera>
           <topic>${camera_sensor_topic}</topic>

File: src/cs625_ap_description/urdf/cs625_parallel_gripper.xacro (robot description, xacro)
@@ -7,8 +7,9 @@
       left   arm  X [-147.31, -27.31]  Y [-9.03, 48.97]  Z [  4.0, 150.0] mm
       right  arm  X [ 113.29, 147.29]  Y [-9.03, 48.97]  Z [  4.0, 150.0] mm
-    each 58 mm deep and 146 mm tall.  What matters for the grasp is the INNER
-    face: the module's handle inner span is 244.00 mm, so with zero interference
-    the arms close on +/-122.00 mm.  Each arm therefore starts retracted at
-    +/-102.00 mm and travels 20 mm outward to the contact plane.
+    each 58 mm deep and 146 mm tall.  What matters for the grasp is the OUTER
+    face of each arm (the surface that presses on a handle's inner face): the
+    module's handle inner span is 244.00 mm, so with zero interference the arms
+    open to +/-122.00 mm.  Each arm therefore starts retracted at +/-102.00 mm
+    and travels outward to the contact plane.
     These are NOT a model of the real linkage.  They are the real contact plane,
     travel direction and cross-section carried by a simplified slab, so the
@@ -17,8 +18,57 @@
       - cs625_active_perception.srdf names these links in disable_collisions,
       - sim_controllers.yaml drives gripper_right_finger_joint,
-      - test/apply_task_fixture_scene.py uses FINGER_LINKS by name.
-    Masses stay at 1 g: the measured 4.580 kg of the tool, mesh included, sits on
-    my_end_effector_link, and these links are its children, so counting them again
-    would double the tool.
+      - test/p7_apply_fixture_scene.py uses FINGER_LINKS by name.
+    TRAVEL (aligned 2026-10-24).  Only two aperture numbers exist for this tool,
+    and both are CAD measurements made by the tool owner, not bench
+    measurements of the assembled gripper:
+      j = 0            outer-face span 204.000 mm   retracted.  NOT MEASURED:
+                                                    the retracted span is a
+                                                    derived value (contact span
+                                                    minus the 20 mm travel), so
+                                                    this end of the range is
+                                                    UNVERIFIED.
+      j = 0.020000     outer-face span 244.000 mm   = the module's measured
+                                                    handle inner span.  This is
+                                                    the zero-preload grasp pose
+                                                    chosen by the task owner
+                                                    (see config/cs625_task_scene.yaml,
+                                                    interference_fit: none_zero_preload).
+      j = 0.021285     outer-face span 246.570 mm   = SolidWorks measured span
+                                                    between the tool's two
+                                                    parallel arm faces
+                                                    (cs625_task_scene.yaml,
+                                                    measured_arm_span_m: 0.24657).
+    Aperture mapping used below, exact for this slab model:
+      span_outer_mm(j) = 204.0 + 2000.0 * j        (j in metres)
+      j(span_outer_mm) = (span_outer_mm - 204.0) / 2000.0
+    The upper limit was 0.020, which is the zero-preload contact, i.e. the model
+    stopped 2.57 mm short of the measured full aperture.  It is now 0.021285 so
+    the joint range reaches the measured span; the grasp itself still commands
+    0.020, and the extra 1.285 mm per side is exactly the real preload that a
+    rigid-body contact deliberately does not apply.
+    STILL NOT ALIGNED, because no number exists to align with: the HITBOT EFG80
+    drive coordinate that config/tasks/common.yaml calls grip_width_mm: 50.0.
+    The drive's position_mm (0..80 command range) is a serial/encoder coordinate,
+    and docs/agent_memory.md section 76 records that this displayed position does
+    NOT equal the physical opening ("归零后有偏移误差，显示位置与实际开度不完全
+    一致").  No log maps drive millimetres to a jaw span, so 50 mm CANNOT be
+    converted into a span here.  Any statement that "the simulator opens to
+    50 mm" would be an invention.  MISSING DATA: measured outer-face span at a
+    set of drive positions (calibration table), plus the retracted span.
+    MASS: ESTIMATED, needs CAD mass/CoG.  These are NOT measured values.
+    my_end_effector_link already carries the MEASURED 4.580 kg of the same rigid
+    body (SolidWorks export 夹持机构0920, see cs625_active_perception.urdf.xacro)
+    and these links sit inside that body, so every kilogram put here is counted
+    twice.  The values below are deliberately small bookkeeping estimates
+    (0.100 + 2 x 0.020 = 0.140 kg, a 3.1% duplicate) whose only job is to give
+    the tree physically sane inertials instead of 1e-9 placeholders.  The
+    physically plausible split still has to come from CAD: a SOLID arm slab of
+    0.055 x 0.058 x 0.146 m at the measured 2.677 g/cm^3 aluminium density would
+    be 1.246 kg (certainly hollow in reality), plus an unknown housing share of
+    the remaining 2.09 kg.  Do not quote the numbers below as the gripper mass;
+    the gripper mass is 4.580 kg and it lives on my_end_effector_link.
+    effort = 80 N and velocity = 0.02 m/s are also UNVERIFIED: the real gripper
+    is run current-limited at 0.1 A (config/tasks/common.yaml grip_current), and
+    no force or speed measurement exists in this repository.
     ZERO INTERFERENCE was chosen deliberately.  The real tool closes with 2.57 mm
     of preload, which a rigid-body contact cannot reproduce honestly: it would
@@ -31,6 +81,10 @@
     <link name="${prefix}gripper_base_link">
       <inertial>
-        <mass value="0.001"/>
-        <inertia ixx="1e-9" ixy="0" ixz="0" iyy="1e-9" iyz="0" izz="1e-9"/>
+        <!-- ESTIMATED, needs CAD mass/CoG.  Not measured.  Bookkeeping share of
+             the 4.580 kg body that already sits on my_end_effector_link; a
+             90 x 90 x 50 mm envelope with the CoM left at the mounting face.
+             Inertia is the solid-box value for 0.100 kg at that envelope. -->
+        <mass value="0.100"/>
+        <inertia ixx="8.83e-05" ixy="0" ixz="0" iyy="8.83e-05" iyz="0" izz="1.35e-04"/>
       </inertial>
     </link>
@@ -52,7 +106,12 @@
       </collision>
       <inertial>
+        <!-- ESTIMATED, needs CAD mass/CoG.  Not measured.  CoM at the slab
+             centre; inertia is the solid-box value for 0.020 kg over
+             0.055 x 0.058 x 0.146 m.  See the MASS note above: 0.020 kg is a
+             bookkeeping duplicate, not the arm's real mass (a solid slab of
+             this size would be 1.246 kg). -->
         <origin xyz="-0.0275 0 0"/>
-        <mass value="0.001"/>
-        <inertia ixx="1e-9" ixy="0" ixz="0" iyy="1e-9" iyz="0" izz="1e-9"/>
+        <mass value="0.020"/>
+        <inertia ixx="4.11e-05" ixy="0" ixz="0" iyy="4.06e-05" iyz="0" izz="1.07e-05"/>
       </inertial>
     </link>
@@ -60,8 +119,9 @@
       <parent link="${prefix}gripper_base_link"/>
       <child link="${prefix}gripper_right_finger_link"/>
-      <!-- Retracted at 102.0 mm; 0.020 m of travel reaches 122.0 mm. -->
+      <!-- Retracted at 102.0 mm; 21.285 mm of travel reaches the measured
+           123.285 mm = 246.57 mm aperture.  0.020 is the zero-preload grasp. -->
       <origin xyz="0.102 0 0.077" rpy="0 0 0"/>
       <axis xyz="1 0 0"/>
-      <limit lower="0.0" upper="0.020" effort="80" velocity="0.02"/>
+      <limit lower="0.0" upper="0.021285" effort="80" velocity="0.02"/>
     </joint>
     <!-- Left arm: mirrored; outer face at joint x = 0, slab extends in +X. -->
@@ -77,7 +137,8 @@
       </collision>
       <inertial>
+        <!-- ESTIMATED, needs CAD mass/CoG.  Mirror of the right arm. -->
         <origin xyz="0.0275 0 0"/>
-        <mass value="0.001"/>
-        <inertia ixx="1e-9" ixy="0" ixz="0" iyy="1e-9" iyz="0" izz="1e-9"/>
+        <mass value="0.020"/>
+        <inertia ixx="4.11e-05" ixy="0" ixz="0" iyy="4.06e-05" iyz="0" izz="1.07e-05"/>
       </inertial>
     </link>
@@ -88,5 +149,5 @@
       <axis xyz="-1 0 0"/>
       <mimic joint="${prefix}gripper_right_finger_joint" multiplier="1.0" offset="0.0"/>
-      <limit lower="0.0" upper="0.020" effort="80" velocity="0.02"/>
+      <limit lower="0.0" upper="0.021285" effort="80" velocity="0.02"/>
     </joint>
     <ros2_control name="${prefix}cs625_parallel_gripper" type="system">
